Commit message: Add Gazebo differential drive simulation

File: description/robot_core.xacro (robot description, xacro)
@@ -41,4 +41,7 @@
         </xacro:inertial_box>
     </link>
+    <gazebo reference="chassi">
+        <material>Gazebo/white</material>
+    </gazebo>
     <!-- left wheel link -->
     <joint name="left_wheel_joint" type="continuous">
@@ -66,4 +69,7 @@
         </xacro:inertial_cylinder>
     </link>
+    <gazebo reference="left_wheel">
+        <material>Gazebo/blue</material>
+    </gazebo>
     <!-- right wheel link -->
     <joint name="right_wheel_joint" type="continuous">
@@ -91,4 +97,7 @@
         </xacro:inertial_cylinder>
     </link>
+    <gazebo reference="right_wheel">
+        <material>Gazebo/blue</material>
+    </gazebo>
     <!-- front caster link -->
     <joint name="front_caster_joint" type="fixed">
@@ -113,3 +122,8 @@
         </xacro:inertial_sphere>
     </link>
+    <gazebo reference="front_caster">
+        <material>Gazebo/black</material>
+        <mu1 value="0.001"/>
+        <mu2 value="0.001"/>
+    </gazebo>
 </robot>

Commit message: Add base footprint frame and fix chassis naming

File: description/robot_core.xacro (robot description, xacro)
@@ -14,14 +14,20 @@
         <color rgba="1 0.3 0.1 1" />
     </material>
-    <!-- Base link -->
-    <link name="base_link">
-    </link>
-    <!-- Chassi link -->
-    <joint name="chassi_joint" type="fixed">
+    <!-- Robot footprint projected onto the ground plane -->
+    <link name="base_footprint"/>
+    <joint name="base_footprint_joint" type="fixed">
+        <parent link="base_footprint"/>
+        <child link="base_link"/>
+        <origin xyz="0 0 0.05" rpy="0 0 0"/>
+    </joint>
+    <!--base link at wheel-center height -->
+    <link name="base_link"/>
+    <!-- chassis link -->
+    <joint name="chassis_joint" type="fixed">
         <parent link="base_link"/>
-        <child link="chassi"/>
+        <child link="chassis"/>
         <origin xyz="-0.1 0 0" />
     </joint>
-    <link name="chassi">
+    <link name="chassis">
         <visual>
             <origin xyz="0.15 0 0.075" />
@@ -41,5 +47,5 @@
         </xacro:inertial_box>
     </link>
-    <gazebo reference="chassi">
+    <gazebo reference="chassis">
         <material>Gazebo/white</material>
     </gazebo>
